File: PoEpi_v2/PoEpi_v2.brd (EAGLE design)
At the start: 88.9 x 58.5 mm, 31 parts, among them IC1 DS2482-100, IC2 MC34063A, IC3 PFC8583P, J1 J25MM, Q1 2N7000, Q2 2N7000

Commit message: Schematics cleanup
Parts:
- Q4: value (none) -> 32.768 kHz
Connections:
- net N$17 renamed +BAT
- removed net N$11: IC1.6
Changed lines of the file:
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@@
 <attribute name="VALUE" x="60.071" y="40.8686" size="1.27" layer="27" ratio="10" rot="R180"/>
 </element>
-<element name="Q4" library="crystal" package="TC26V" value="" x="63.5" y="31.75" rot="R270">
+<element name="Q4" library="crystal" package="TC26V" value="32.768 kHz" x="63.5" y="31.75" rot="R270">
 <attribute name="OC_NEWARK" value="unknown" x="63.5" y="31.75" size="1.778" layer="27" rot="R270" display="off"/>
 <attribute name="MPN" value="" x="63.5" y="31.75" size="1.778" layer="27" rot="R270" display="off"/>
@@
 <contactref element="C2" pad="-"/>
 <contactref element="R4" pad="2"/>
-<contactref element="IC2" pad="4"/>
 <contactref element="C3" pad="2"/>
-<contactref element="IC2" pad="4"/>
-<contactref element="D1" pad="A"/>
 <contactref element="B1" pad="-"/>
 <wire x1="50.165" y1="15.24" x2="48.26" y2="15.24" width="0.4064" layer="16"/>
@@
 <wire x1="3.81" y1="40.64" x2="1.27" y2="40.64" width="0.6096" layer="16"/>
 <wire x1="1.27" y1="40.64" x2="1.27" y2="48.26" width="0.6096" layer="16"/>
-<wire x1="3.81" y1="40.64" x2="7.62" y2="40.64" width="0.6096" layer="16"/>
 <wire x1="48.26" y1="12.7" x2="48.26" y2="15.24" width="0.4064" layer="16"/>
 <wire x1="78.105" y1="55.88" x2="49.53" y2="55.88" width="0.6096" layer="16"/>
 <wire x1="49.53" y1="55.88" x2="27.94" y2="55.88" width="0.6096" layer="16"/>
 <wire x1="27.94" y1="55.88" x2="3.81" y2="55.88" width="0.6096" layer="16"/>
-<wire x1="3.81" y1="55.88" x2="3.81" y2="52.07" width="0.6096" layer="16"/>
 <wire x1="40.1066" y1="45.085" x2="41.91" y2="45.085" width="0.4064" layer="16"/>
 <wire x1="41.91" y1="45.085" x2="41.91" y2="43.815" width="0.4064" layer="16"/>
@@
 <wire x1="49.53" y1="48.26" x2="49.53" y2="55.88" width="0.4064" layer="16"/>
 <wire x1="27.94" y1="53.213" x2="27.94" y2="55.88" width="0.6096" layer="16"/>
-<wire x1="3.81" y1="52.07" x2="3.81" y2="48.26" width="0.6096" layer="16"/>
 <wire x1="3.81" y1="48.26" x2="1.27" y2="48.26" width="0.6096" layer="16"/>
 <wire x1="5.08" y1="48.26" x2="3.81" y2="48.26" width="0.4064" layer="16"/>
@@
 <wire x1="43.18" y1="21.59" x2="43.18" y2="12.7" width="0.4064" layer="16"/>
 <wire x1="43.18" y1="12.7" x2="48.26" y2="12.7" width="0.4064" layer="16"/>
+<contactref element="IC2" pad="4"/>
+<contactref element="D1" pad="A"/>
+<contactref element="IC2" pad="4"/>
+<wire x1="7.62" y1="40.64" x2="3.81" y2="40.64" width="0.6096" layer="16"/>
+<wire x1="3.81" y1="52.07" x2="3.81" y2="48.26" width="0.6096" layer="16"/>
+<wire x1="3.81" y1="52.07" x2="3.81" y2="55.88" width="0.6096" layer="16"/>
 </signal>
 <signal name="TXD">
@@
 <wire x1="48.895" y1="21.59" x2="48.895" y2="17.78" width="0.4064" layer="16"/>
 </signal>
-<signal name="N$11">
-<contactref element="IC1" pad="6"/>
-</signal>
 <signal name="N$14">
 <contactref element="B1" pad="AC2"/>
@@
 <wire x1="50.8" y1="29.21" x2="53.34" y2="29.21" width="0.4064" layer="16"/>
 </signal>
-<signal name="N$17">
+<signal name="+BAT">
 <contactref element="G1" pad="+"/>
 <contactref element="G1" pad="+@1"/>
@@
 </signal>
 </signals>
+<errors>
+</errors>
 </board>
 </drawing>
