File: PoEpi_v2/PoEpi_v2.sch (EAGLE design)
At the start: 31 parts, among them IC1 DS2482-100, IC2 MC34063A, IC3 PFC8583P, J1 J25MM, Q1 2N7000, Q2 2N7000

Commit message: Schematics cleanup
Parts:
- Q4: value (none) -> 32.768 kHz
Connections:
- net N$17 renamed +BAT
- removed net N$11: IC1.PCTLZ
Other:
- moved on the sheet: C1, C2, D1, F1, L1, Q1, TP2
